Commit message: pybullet sim

File: assets/foam-2.urdf (robot description, URDF)
Before this commit: robot physics, 2 links, 1 joints
Links:
- added link link2; collision mesh filename=unit.stl scale=0.1 0.1 0.1; visual mesh filename=unit.stl scale=0.1 0.1 0.1
- link base_link: geometry collision mesh filename=unit.stl scale=0.1 0.1 0.1; visual mesh filename=unit.stl scale=0.1 0.1 0.1
- link link1: geometry collision mesh filename=unit.stl scale=0.1 0.1 0.1; visual mesh filename=unit.stl scale=0.1 0.1 0.1
Joints:
- added joint joint12: type revolute, parent link1, child link2, origin xyz=2.5 0 0, axis 0 1 0, limit lower=-1 effort=300 velocity=1
- joint joint01: limit effort=300 velocity=1 -> lower=-1 effort=300 velocity=1

Commit message: grasp sim

File: assets/foam-2.urdf (robot description, URDF)
Before this commit: robot physics, 3 links, 2 joints
Links:
- link base_link: mass None -> .5
- link link1: mass None -> .5
- link link2: mass None -> .5
Joints:
- joint joint01: limit lower=-1 effort=300 velocity=1 -> lower=-1.3 effort=300 velocity=1
- joint joint12: limit lower=-1 effort=300 velocity=1 -> lower=-1.3 effort=300 velocity=1
