Commit message: gripper model

File: assets/cube.urdf (robot description, URDF)
Before this commit: robot cube, 1 links, 0 joints
Links:
- link base_link: mass 5 -> None; geometry collision mesh filename=Cube.stl scale=0.001 0.001 0.001; visual mesh filename=Cube.stl scale=0.001 0.001 0.001

File: assets/foam-2.urdf (robot description, URDF)
Before this commit: robot physics, 3 links, 2 joints
Links:
- link base_link: mass .5 -> None; geometry collision mesh filename=unit.stl scale=0.001 0.001 0.001; visual mesh filename=unit.stl scale=0.001 0.001 0.001
- link link1: mass .5 -> None; geometry collision mesh filename=unit.stl scale=0.001 0.001 0.001; visual mesh filename=unit.stl scale=0.001 0.001 0.001
- link link2: mass .5 -> None; geometry collision mesh filename=unit.stl scale=0.001 0.001 0.001; visual mesh filename=unit.stl scale=0.001 0.001 0.001
Joints:
- joint joint01: limit lower=-1.3 effort=300 velocity=1 -> lower=-.1 upper=1.3 effort=300 velocity=1; origin xyz=2.25 0 0 -> xyz=0.0225 0 0
- joint joint12: limit lower=-1.3 effort=300 velocity=1 -> lower=-.1 upper=1.3 effort=300 velocity=1; origin xyz=2.5 0 0 -> xyz=0.025 0 0
